Commit message: driving virtual robot

File: description/robot_core.xacro (robot description, xacro)
@@ -29,5 +29,5 @@
                     <box size="0.3 0.3 0.15"/>
                 </geometry>
-                <material name="white"/>
+                <material name="blue"/>
             </visual>
             <collision>
@@ -41,4 +41,7 @@
             </xacro:inertial_box>
         </link>
+        <gazebo reference="chassis">
+            <material>Gazebo/Blue</material>
+        </gazebo>
           <!-- LEFT WHEEL LINK -->
     <joint name="left_wheel_joint" type="continuous">
@@ -53,5 +56,5 @@
                 <cylinder radius="0.05" length="0.04"/>
             </geometry>
-            <material name="blue"/>
+            <material name="black"/>
         </visual>
         <collision>
@@ -64,4 +67,7 @@
         </xacro:inertial_cylinder>
     </link>
+    <gazebo reference="left_wheel">
+        <material>Gazebo/Black</material>
+    </gazebo>
             <!-- RIGHT WHEEL LINK -->
     <joint name="right_wheel_joint" type="continuous">
@@ -76,5 +82,5 @@
                 <cylinder radius="0.05" length="0.04"/>
             </geometry>
-            <material name="blue"/>
+            <material name="black"/>
         </visual>
         <collision>
@@ -87,4 +93,7 @@
         </xacro:inertial_cylinder>
     </link>
+    <gazebo reference="right_wheel">
+        <material>Gazebo/Black</material>
+    </gazebo>
       <!-- CASTER WHEEL LINK -->
       <joint name="caster_wheel_joint" type="fixed">
@@ -98,5 +107,5 @@
                 <sphere radius="0.05"/>
             </geometry>
-            <material name="black"/>
+            <material name="white"/>
         </visual>
         <collision>
@@ -109,3 +118,8 @@
         </xacro:inertial_sphere>
     </link>
+    <gazebo reference="caster_wheel">
+        <material>Gazebo/White</material>
+        <mu1 value="0.001"/>
+        <mu2 value="0.001"/>
+    </gazebo>
 </robot>
