Commit message: SLAM with ROS using slam_toolbox

File: description/lidar.xacro (robot description, xacro)
@@ -23,5 +23,5 @@
     </link>
     <gazebo reference="laser_frame">
-        <material>Gazebo/Red</material>
+        <material>Gazebo/red</material>
         <sensor name="laser" type="ray">
             <pose> 0 0 0 0 0 0 </pose>

File: description/robot.urdf.xacro (robot description, xacro)
@@ -1,6 +1,12 @@
 <?xml version="1.0"?>
 <robot xmlns:xacro="http://www.ros.org/wiki/xacro"  name="robot">
+    <xacro:arg name="use_ros2_control" default="true" />
     <xacro:include filename="robot_core.xacro" />
-    <xacro:include filename="gazebo_control.xacro" />
+    <xacro:if value="$(arg use_ros2_control)">
+        <xacro:include filename="ros2_control.xacro" />
+    </xacro:if>
+    <xacro:unless value="$(arg use_ros2_control)">
+        <xacro:include filename="gazebo_control.xacro" />
+    </xacro:unless>
     <xacro:include filename="lidar.xacro" />
     <!-- <xacro:include filename="camera.xacro" /> -->

File: description/robot_core.xacro (robot description, xacro)
@@ -11,4 +11,7 @@
         <color rgba="0.2 0.2 1 1"/>
     </material>
+    <material name="red">
+        <color rgba="1 0 0 1"/>
+    </material>
     <material name="black">
         <color rgba="0 0 0 1"/>
@@ -16,4 +19,12 @@
         <!-- BASE LINK -->
         <link name="base_link">
+        </link>
+        <!-- Base_FOOTPRINT LINK -->
+        <joint name="base_footprint_joint" type="fixed">
+            <parent link="base_link"/>
+            <child link="base_footprint"/>
+            <origin xyz="0 0 0" rpy="0 0 0"/>
+        </joint>
+        <link name="base_footprint">
         </link>
         <!-- CHASSIS LINK -->
